Commit message: nav2

File: workspace/src/c_megarover_description/urdf/mega3_base_model.xacro (robot description, xacro)
@@ -5,7 +5,7 @@
   <link name="base_footprint" />
   <joint name="base_joint" type="fixed">
-    <parent link="base_footprint" />
-    <child link="base_link" />
-    <origin xyz="-0.1 0 0" rpy="0 0 -1.5708" />
+    <origin xyz="0 0 0"/>
+    <parent link="base_footprint"/>
+    <child link="base_link"/>
   </joint>
   <link name="base_link">

File: workspace/src/c_megarover_description/urdf/mega3_lidar.xacro (robot description, xacro)
@@ -27,5 +27,5 @@
         <parent link="base_link" />
         <child link="livox_frame" />
-        <origin xyz="0 0.1 0.2" rpy="0 0 1.5708" />
+        <origin xyz="0 0.1 0.2" rpy="0 0 0" />
     </joint>
 </robot>

Commit message: update

File: workspace/src/c_megarover_description/urdf/mega3_base_model.xacro (robot description, xacro)
@@ -1,5 +1,5 @@
 <?xml version="1.0"?>
 <robot name="mega3" xmlns:xacro="http://www.ros.org/wiki/xacro">
-  <xacro:include filename="$(find megarover_description)/urdf/materials.xacro" />
+  <xacro:include filename="$(find c_megarover_description)/urdf/materials.xacro" />
   <!-- <xacro:include filename="$(find megarover_description)/urdf/mega3_base_model.gazebo" /> -->
   <link name="base_footprint" />
@@ -11,5 +11,5 @@
   <link name="base_link">
     <inertial>
-      <origin xyz="-0.0001512201285105937 -3.420007213019073e-05 0.08388833658828038" rpy="0 0 0" />
+      <origin xyz="0 0 0" rpy="0 0 0" />
       <mass value="11.744482" />
       <inertia ixx="0.091465" iyy="0.06435" izz="0.1253"
@@ -20,17 +20,17 @@
       <origin xyz="0 0 0" rpy="0 0 0" />
       <geometry>
-        <mesh filename="$(find megarover_description)/meshes/mega3/base_link.stl" scale="0.001 0.001 0.001" />
+        <mesh filename="package://c_megarover_description/meshes/mega3/base_link_v3.stl" scale="0.0001 0.0001 0.0001" />
       </geometry>
       <material name="silver" />
     </visual>
     <collision>
-      <origin xyz="0 0 0" rpy="0 0 0" />
+      <origin xyz="0 0 0" rpy="0 0 0"/>
       <geometry>
-        <mesh filename="$(find megarover_description)/meshes/mega3/base_link.stl" scale="0.001 0.001 0.001" />
+        <mesh filename="package://c_megarover_description/meshes/mega3/base_link_v3.stl" scale="0.0001 0.0001 0.0001" />
       </geometry>
     </collision>
   </link>
   <joint name="left_wheel_joint" type="continuous">
-    <origin xyz="-0.136 0.1 0.07" rpy="0 -1.5708 0" />
+    <origin xyz="0.1 0.136 0.07" rpy="-1.57 0 0" />
     <parent link="base_link" />
     <child link="left_wheel_1" />
@@ -39,5 +39,5 @@
   <link name="left_wheel_1">
     <inertial>
-      <origin xyz="0.0 0.0 0.00213" rpy="0 1.5708 0" />
+      <origin xyz="0 0 0" rpy="1.57 0 0" />
       <mass value="1.239934" />
       <inertia ixx="0.002474" iyy="0.00174" izz="0.00174"
@@ -46,19 +46,19 @@
     </inertial>
     <visual>
-      <origin xyz="-0.07 -0.1 -0.136" rpy="0 1.5708 0" />
+      <origin xyz="0 0 0" rpy="1.57 0 0" />
       <geometry>
-        <mesh filename="$(find megarover_description)/meshes/mega3/left_wheel_1.stl" scale="0.001 0.001 0.001" />
+        <mesh filename="package://c_megarover_description/meshes/mega3/left_wheel_1_v3.stl" scale="0.001 0.001 0.001" />
       </geometry>
       <material name="dark_grey" />
     </visual>
     <collision>
-      <origin xyz="-0.07 -0.1 -0.136" rpy="0 1.5708 0" />
+      <origin xyz="0 0 0" rpy="1.57 0 0" />
       <geometry>
-        <mesh filename="$(find megarover_description)/meshes/mega3/left_wheel_1.stl" scale="0.001 0.001 0.001" />
+        <mesh filename="package://c_megarover_description/meshes/mega3/left_wheel_1_v3.stl" scale="0.001 0.001 0.001" />
       </geometry>
     </collision>
   </link>
   <joint name="right_wheel_joint" type="continuous">
-    <origin xyz="0.136 0.1 0.07" rpy="0 -1.5708 0" />
+    <origin xyz="0.1 -0.136 0.07" rpy="-1.57 0 0" />
     <parent link="base_link" />
     <child link="right_wheel_1" />
@@ -67,5 +67,5 @@
   <link name="right_wheel_1">
     <inertial>
-      <origin xyz="0 0 -0.00213" rpy="0 1.5708 0" />
+      <origin xyz="0 0 0" rpy="1.57 0 0" />
       <mass value="1.239934" />
       <inertia ixx="0.002474" iyy="0.00174" izz="0.00174"
@@ -74,7 +74,7 @@
     </inertial>
     <visual>
-      <origin xyz="-0.07 -0.1 0.136" rpy="0 1.5708 0" />
+      <origin xyz="0 0 0" rpy="1.57 0 0" />
       <geometry>
-        <mesh filename="$(find megarover_description)/meshes/mega3/right_wheel_1.stl" scale="0.001 0.001 0.001" />
+        <mesh filename="package://c_megarover_description/meshes/mega3/right_wheel_1_v3.stl" scale="0.001 0.001 0.001" />
       </geometry>
       <material name="dark_grey" />
@@ -83,5 +83,5 @@
       <origin xyz="-0.07 -0.1 0.136" rpy="0 1.5708 0" />
       <geometry>
-        <mesh filename="$(find megarover_description)/meshes/mega3/right_wheel_1.stl" scale="0.001 0.001 0.001" />
+        <mesh filename="package://c_megarover_description/meshes/mega3/right_wheel_1_v3.stl" scale="0.001 0.001 0.001" />
       </geometry>
     </collision>

File: workspace/src/c_megarover_description/urdf/mega3_lidar.xacro (robot description, xacro)
@@ -27,5 +27,5 @@
         <parent link="base_link" />
         <child link="livox_frame" />
-        <origin xyz="0 0.1 0.2" rpy="0 0 0" />
+        <origin xyz="0.15 0 0.2" rpy="0 0 0" />
     </joint>
     <!-- For FAST_LIO -->
@@ -34,5 +34,5 @@
         <parent link="base_link" />
         <child link="camera_init" />
-        <origin xyz="0 0.1 0.2" rpy="0 0 0" />
+        <origin xyz="0.15 0 0.2" rpy="0 0 0" />
     </joint>
 </robot>

Commit message: update

File: workspace/src/c_megarover_description/urdf/mega3_base_model.xacro (robot description, xacro)
@@ -20,5 +20,5 @@
       <origin xyz="0 0 0" rpy="0 0 0" />
       <geometry>
-        <mesh filename="package://c_megarover_description/meshes/mega3/base_link_v3.stl" scale="0.0001 0.0001 0.0001" />
+        <mesh filename="package://c_megarover_description/meshes/mega3/base_link_v5.stl" scale="0.001 0.001 0.001" />
       </geometry>
       <material name="silver" />
@@ -27,5 +27,5 @@
       <origin xyz="0 0 0" rpy="0 0 0"/>
       <geometry>
-        <mesh filename="package://c_megarover_description/meshes/mega3/base_link_v3.stl" scale="0.0001 0.0001 0.0001" />
+        <mesh filename="package://c_megarover_description/meshes/mega3/base_link_v5.stl" scale="0.001 0.001 0.001" />
       </geometry>
     </collision>
