Commit message: update

File: workspace/src/c_megarover_description/urdf/mega3_lidar.xacro (robot description, xacro)
@@ -27,5 +27,5 @@
         <parent link="base_link" />
         <child link="livox_frame" />
-        <origin xyz="0 0.1 0.2" rpy="0 0 0" />
+        <origin xyz="0 0.1 0.2" rpy="0 0 1.5708" />
     </joint>
 </robot>

Commit message: add

File: workspace/src/c_megarover_description/urdf/mega3_lidar.xacro (robot description, xacro)
@@ -29,3 +29,10 @@
         <origin xyz="0 0.1 0.2" rpy="0 0 0" />
     </joint>
+    <!-- For FAST_LIO -->
+    <link name="camera_init" />
+    <joint name="camera_init_joint" type="fixed">
+        <parent link="livox_frame" />
+        <child link="camera_init" />
+        <origin xyz="0 0 0" rpy="0 0 0" />
+    </joint>
 </robot>

Commit message: update

File: workspace/src/c_megarover_description/urdf/mega3_lidar.xacro (robot description, xacro)
@@ -32,7 +32,7 @@
     <link name="camera_init" />
     <joint name="camera_init_joint" type="fixed">
-        <parent link="livox_frame" />
+        <parent link="base_link" />
         <child link="camera_init" />
-        <origin xyz="0 0 0" rpy="0 0 0" />
+        <origin xyz="0 0.1 0.2" rpy="0 0 0" />
     </joint>
 </robot>

Commit message: update

File: workspace/src/c_megarover_description/urdf/mega3_lidar.xacro (robot description, xacro)
@@ -27,5 +27,5 @@
         <parent link="base_link" />
         <child link="livox_frame" />
-        <origin xyz="0.15 0 0.2" rpy="0 0 0" />
+        <origin xyz="0.15 0 0.60" rpy="0 0 0" />
     </joint>
     <!--

Commit message: update

File: workspace/src/c_megarover_description/urdf/mega3_lidar.xacro (robot description, xacro)
@@ -27,5 +27,5 @@
         <parent link="base_link" />
         <child link="livox_frame" />
-        <origin xyz="0.15 0 0.60" rpy="0 0 0" />
+        <origin xyz="0.15 0 0.65" rpy="0 0 0" />
     </joint>
     <!--
